File: eagle/coildriver/Driver3.brd (EAGLE design)
At the start: 99.1 x 63.5 mm, 43 parts, among them IC1 7905L, Q1 BC327, Q2 BC327, Q3 IGBT

Commit message: Silkscreen fixes
Parts:
- R13: value 620 -> 620R
Changed lines of the file:
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@@
 <text x="70.485" y="15.875" size="1.27" layer="51" rot="R270">+12V</text>
 <text x="65.405" y="15.875" size="1.27" layer="51" rot="R270">GND</text>
-<text x="66.675" y="46.99" size="1.27" layer="51" rot="R90">COIL -</text>
-<text x="71.755" y="46.99" size="1.27" layer="51" rot="R90">COIL +</text>
+<text x="71.755" y="46.99" size="1.27" layer="51" rot="R90">COIL -</text>
+<text x="66.675" y="46.99" size="1.27" layer="51" rot="R90">COIL +</text>
 <text x="90.17" y="50.165" size="1.016" layer="52" font="vector" rot="MR0">Licensed under the TAPR NCL</text>
 <text x="85.09" y="47.625" size="1.016" layer="52" font="vector" rot="MR0">www.tapr.org/NCL</text>
@@
 <attribute name="VALUE" x="10.16" y="6.985" size="1.27" layer="27" font="fixed"/>
 </element>
-<element name="R13" library="resistor" package="0204/7" value="620" x="17.78" y="12.7" rot="R90"/>
+<element name="R13" library="resistor" package="0204/7" value="620R" x="17.78" y="12.7" rot="R90"/>
 <element name="FREQ" library="pinhead" package="1X02" value="FREQ" x="24.13" y="12.7" smashed="yes" rot="R180">
 <attribute name="NAME" x="26.7462" y="10.8712" size="1.27" layer="25" ratio="10" rot="R180"/>
