File: eagle/coildriver/Driver3.sch (EAGLE design)
At the start: 43 parts, among them IC1 7905L, Q1 BC327, Q2 BC327, Q3 IGBT

Commit message: Silkscreen fixes
Parts:
- R13: value 620 -> 620R
Changed lines of the file:
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@@
 <part name="R9" library="resistor" deviceset="R-US_" device="0204/7" value="100K"/>
 <part name="OPTO-IN" library="pinhead" deviceset="PINHD-1X2" device="" value="OPTO-IN"/>
-<part name="R13" library="resistor" deviceset="R-US_" device="0204/7" value="620"/>
+<part name="R13" library="resistor" deviceset="R-US_" device="0204/7" value="620R"/>
 <part name="FREQ" library="pinhead" deviceset="PINHD-1X2" device="" value="FREQ"/>
 <part name="R1" library="resistor" deviceset="R-US_" device="0204/7" value="620R"/>
